Commit message: integration of hybrid control with cartesian space and joint space

File: src/DESCRIPTION/cerberus_v1/description/roscon/template_roscon.xacro (robot description, xacro)
@@ -17,5 +17,5 @@
                 <param name="initial_position">0.0</param>
                 <param name="max_velocity">5.8178</param>
-                <param name="max_effort">1.7</param>
+                <param name="max_effort">1.67</param>
             </joint>
             <joint name="ThFR_SeFR">
@@ -31,5 +31,5 @@
                 <param name="initial_position">0.0</param>
                 <param name="max_velocity">5.8178</param>
-                <param name="max_effort">1.7</param>
+                <param name="max_effort">1.67</param>
             </joint>
             <joint name="ArFR_ThFR">
@@ -45,5 +45,5 @@
                 <param name="initial_position">0.0</param>
                 <param name="max_velocity">5.8178</param>
-                <param name="max_effort">1.7</param>
+                <param name="max_effort">1.67</param>
             </joint>
             <joint name="ShFR_ThFR" mimic="${enable_mimic}">
@@ -61,5 +61,5 @@
                 <param name="initial_position">0.0</param>
                 <param name="max_velocity">5.8178</param>
-                <param name="max_effort">1.7</param>
+                <param name="max_effort">1.67</param>
                 <param name="mimic">ArFR_ThFR</param>
                 <param name="multiplier">-0.2824</param>
@@ -79,5 +79,5 @@
                 <param name="initial_position">0.0</param>
                 <param name="max_velocity">5.8178</param>
-                <param name="max_effort">1.7</param>
+                <param name="max_effort">1.67</param>
             </joint>
             <joint name="ThFL_SeFL">
@@ -93,5 +93,5 @@
                 <param name="initial_position">0.0</param>
                 <param name="max_velocity">5.8178</param>
-                <param name="max_effort">1.7</param>
+                <param name="max_effort">1.67</param>
             </joint>
             <joint name="ArFL_ThFL">
@@ -107,5 +107,5 @@
                 <param name="initial_position">0.0</param>
                 <param name="max_velocity">5.8178</param>
-                <param name="max_effort">1.7</param>
+                <param name="max_effort">1.67</param>
             </joint>
             <joint name="ShFL_ThFL" mimic="${enable_mimic}">
@@ -123,5 +123,5 @@
                 <param name="initial_position">0.0</param>
                 <param name="max_velocity">5.8178</param>
-                <param name="max_effort">1.7</param>
+                <param name="max_effort">1.67</param>
                 <param name="mimic">ArFL_ThFL</param>
                 <param name="multiplier">-0.2824</param>
@@ -141,5 +141,5 @@
                 <param name="initial_position">0.0</param>
                 <param name="max_velocity">5.8178</param>
-                <param name="max_effort">1.7</param>
+                <param name="max_effort">1.67</param>
             </joint>
             <joint name="ThBR_SeBR">
@@ -155,5 +155,5 @@
                 <param name="initial_position">0.0</param>
                 <param name="max_velocity">5.8178</param>
-                <param name="max_effort">1.7</param>
+                <param name="max_effort">1.67</param>
             </joint>
             <joint name="ArBR_ThBR">
@@ -169,5 +169,5 @@
                 <param name="initial_position">0.0</param>
                 <param name="max_velocity">5.8178</param>
-                <param name="max_effort">1.7</param>
+                <param name="max_effort">1.67</param>
             </joint>
             <joint name="ShBR_ThBR" mimic="${enable_mimic}">
@@ -185,5 +185,5 @@
                 <param name="initial_position">0.0</param>
                 <param name="max_velocity">5.8178</param>
-                <param name="max_effort">1.7</param>
+                <param name="max_effort">1.67</param>
                 <param name="mimic">ArBR_ThBR</param>
                 <param name="multiplier">-0.2824</param>
@@ -203,5 +203,5 @@
                 <param name="initial_position">0.0</param>
                 <param name="max_velocity">5.8178</param>
-                <param name="max_effort">1.7</param>
+                <param name="max_effort">1.67</param>
             </joint>
             <joint name="ThBL_SeBL">
@@ -217,5 +217,5 @@
                 <param name="initial_position">0.0</param>
                 <param name="max_velocity">5.8178</param>
-                <param name="max_effort">1.7</param>
+                <param name="max_effort">1.67</param>
             </joint>
             <joint name="ArBL_ThBL">
@@ -231,5 +231,5 @@
                 <param name="initial_position">0.0</param>
                 <param name="max_velocity">5.8178</param>
-                <param name="max_effort">1.7</param>
+                <param name="max_effort">1.67</param>
             </joint>
             <joint name="ShBL_ThBL" mimic="${enable_mimic}">
@@ -247,5 +247,5 @@
                 <param name="initial_position">0.0</param>
                 <param name="max_velocity">5.8178</param>
-                <param name="max_effort">1.7</param>
+                <param name="max_effort">1.67</param>
                 <param name="mimic">ArBL_ThBL</param>
                 <param name="multiplier">-0.2824</param>

File: src/DESCRIPTION/cerberus_v1/description/urdf/CERBERUS_V1.urdf (robot description, URDF)
Before this commit: robot CERBERUS_V1, 29 links, 28 joints
Joints:
- joint ArBL_ThBL: limit lower=-0.785398163397 upper=0.785398163397 effort=1.67 velocity=5.0 -> lower=-0.785398163397 upper=0.785398163397 effort=1.67 velocity=5.8178
- joint ArBR_ThBR: limit lower=-0.785398163397 upper=0.785398163397 effort=1.67 velocity=5.0 -> lower=-0.785398163397 upper=0.785398163397 effort=1.67 velocity=5.8178
- joint ArFL_ThFL: limit lower=-0.785398163397 upper=0.785398163397 effort=1.67 velocity=5.0 -> lower=-0.785398163397 upper=0.785398163397 effort=1.67 velocity=5.8178
- joint ArFR_ThFR: limit lower=-0.785398163397 upper=0.785398163397 effort=1.67 velocity=5.0 -> lower=-0.785398163397 upper=0.785398163397 effort=1.67 velocity=5.8178
- joint SeBL_M: limit lower=-0.785398163397 upper=0.785398163397 effort=1.67 velocity=5.0 -> lower=-0.785398163397 upper=0.785398163397 effort=1.67 velocity=5.8178
- joint SeBR_M: limit lower=-0.785398163397 upper=0.785398163397 effort=1.67 velocity=5.0 -> lower=-0.785398163397 upper=0.785398163397 effort=1.67 velocity=5.8178
- joint SeFL_M: limit lower=-0.785398163397 upper=0.785398163397 effort=1.67 velocity=5.0 -> lower=-0.785398163397 upper=0.785398163397 effort=1.67 velocity=5.8178
- joint SeFR_M: limit lower=-0.785398163397 upper=0.785398163397 effort=1.67 velocity=5.0 -> lower=-0.785398163397 upper=0.785398163397 effort=1.67 velocity=5.8178
- joint ShBL_ThBL: limit lower=-0.785398163397 upper=0.785398163397 effort=1.67 velocity=5.0 -> lower=-0.785398163397 upper=0.785398163397 effort=1.67 velocity=5.8178; mimic joint=ArBL_ThBL multiplier=-0.304 offset=0 -> joint=ArBL_ThBL multiplier=-0.2824 offset=0; origin xyz=-0.18101 0.0059195 0.01015 rpy=0 0 1.3090 -> xyz=-0.18101 0.0059195 0.01015 rpy=0 0 1.134
- joint ShBR_ThBR: limit lower=-0.785398163397 upper=0.785398163397 effort=1.67 velocity=5.0 -> lower=-0.785398163397 upper=0.785398163397 effort=1.67 velocity=5.8178; mimic joint=ArBR_ThBR multiplier=-0.304 offset=0 -> joint=ArBR_ThBR multiplier=-0.2824 offset=0; origin xyz=0.18101 0.0059195 0.01015 rpy=0 0 -1.3090 -> xyz=0.18101 0.0059195 0.01015 rpy=0 0 -1.134
- joint ShFL_ThFL: limit lower=-0.785398163397 upper=0.785398163397 effort=1.67 velocity=5.0 -> lower=-0.785398163397 upper=0.785398163397 effort=1.67 velocity=5.8178; mimic joint=ArFL_ThFL multiplier=-0.304 offset=0 -> joint=ArFL_ThFL multiplier=-0.2824 offset=0; origin xyz=-0.18101 0.0059195 0.01015 rpy=0 0 1.3090 -> xyz=-0.18101 0.0059195 0.01015 rpy=0 0 1.134
- joint ShFR_ThFR: limit lower=-0.785398163397 upper=0.785398163397 effort=1.67 velocity=5.0 -> lower=-0.785398163397 upper=0.785398163397 effort=1.67 velocity=5.8178; mimic joint=ArFR_ThFR multiplier=-0.304 offset=0 -> joint=ArFR_ThFR multiplier=-0.2824 offset=0; origin xyz=0.18101 0.0059195 0.01015 rpy=0 0 -1.3090 -> xyz=0.18101 0.0059195 0.01015 rpy=0 0 -1.134
- joint ThBL_SeBL: limit lower=-0.785398163397 upper=0.785398163397 effort=1.67 velocity=5.0 -> lower=-0.785398163397 upper=0.785398163397 effort=1.67 velocity=5.8178
- joint ThBR_SeBR: limit lower=-0.785398163397 upper=0.785398163397 effort=1.67 velocity=5.0 -> lower=-0.785398163397 upper=0.785398163397 effort=1.67 velocity=5.8178
- joint ThFL_SeFL: limit lower=-0.785398163397 upper=0.785398163397 effort=1.67 velocity=5.0 -> lower=-0.785398163397 upper=0.785398163397 effort=1.67 velocity=5.8178
- joint ThFR_SeFR: limit lower=-0.785398163397 upper=0.785398163397 effort=1.67 velocity=5.0 -> lower=-0.785398163397 upper=0.785398163397 effort=1.67 velocity=5.8178
