Commit message: integration of hybrid control with cartesian space and joint space

File: src/DESCRIPTION/cerberus_v1/description/roscon/template_roscon.xacro (robot description, xacro)
@@ -8,13 +8,13 @@
                 <state_interface name="position" />
                 <command_interface name="position">
-                    <param name="min">-0.785398163</param>
-                    <param name="max">0.785398163397</param>
-                </command_interface>
-                <!-- <command_interface name="velocity">
-                    <param name="min">0.0</param>
-                    <param name="max">5.8178</param>
-                </command_interface> -->
-                <param name="initial_position">0.0</param>
-                <param name="max_velocity">5.8178</param>
+                    <param name="min">-0.7854</param>
+                    <param name="max">0.7854</param>
+                </command_interface>
+                <!-- <command_interface name="velocity">
+                    <param name="min">0.0</param>
+                    <param name="max">6.545</param>
+                </command_interface> -->
+                <param name="initial_position">0.0</param>
+                <param name="max_velocity">6.545</param>
                 <param name="max_effort">1.7</param>
             </joint>
@@ -22,13 +22,13 @@
                 <state_interface name="position" />
                 <command_interface name="position">
-                    <param name="min">-0.785398163</param>
-                    <param name="max">0.785398163397</param>
-                </command_interface>
-                <!-- <command_interface name="velocity">
-                    <param name="min">0.0</param>
-                    <param name="max">5.8178</param>
-                </command_interface> -->
-                <param name="initial_position">0.0</param>
-                <param name="max_velocity">5.8178</param>
+                    <param name="min">-0.7854</param>
+                    <param name="max">0.7854</param>
+                </command_interface>
+                <!-- <command_interface name="velocity">
+                    <param name="min">0.0</param>
+                    <param name="max">6.545</param>
+                </command_interface> -->
+                <param name="initial_position">0.0</param>
+                <param name="max_velocity">6.545</param>
                 <param name="max_effort">1.7</param>
             </joint>
@@ -36,13 +36,13 @@
                 <state_interface name="position" />
                 <command_interface name="position">
-                    <param name="min">-0.785398163</param>
-                    <param name="max">0.785398163397</param>
-                </command_interface>
-                <!-- <command_interface name="velocity">
-                    <param name="min">0.0</param>
-                    <param name="max">5.8178</param>
-                </command_interface> -->
-                <param name="initial_position">0.0</param>
-                <param name="max_velocity">5.8178</param>
+                    <param name="min">-0.7854</param>
+                    <param name="max">0.7854</param>
+                </command_interface>
+                <!-- <command_interface name="velocity">
+                    <param name="min">0.0</param>
+                    <param name="max">6.545</param>
+                </command_interface> -->
+                <param name="initial_position">0.0</param>
+                <param name="max_velocity">6.545</param>
                 <param name="max_effort">1.7</param>
             </joint>
@@ -51,14 +51,14 @@
                 <xacro:unless value="${enable_mimic}">
                     <command_interface name="position">
-                        <param name="min">-0.785398163</param>
-                        <param name="max">0.785398163397</param>
-                    </command_interface>
-                    <!-- <command_interface name="velocity">
-                        <param name="min">0.0</param>
-                        <param name="max">5.8178</param>
-                    </command_interface> -->
-                </xacro:unless>
-                <param name="initial_position">0.0</param>
-                <param name="max_velocity">5.8178</param>
+                        <param name="min">-0.7854</param>
+                        <param name="max">0.7854</param>
+                    </command_interface>
+                    <!-- <command_interface name="velocity">
+                        <param name="min">0.0</param>
+                        <param name="max">6.545</param>
+                    </command_interface> -->
+                </xacro:unless>
+                <param name="initial_position">0.0</param>
+                <param name="max_velocity">6.545</param>
                 <param name="max_effort">1.7</param>
                 <param name="mimic">ArFR_ThFR</param>
@@ -70,13 +70,13 @@
                 <state_interface name="position" />
                 <command_interface name="position">
-                    <param name="min">-0.785398163</param>
-                    <param name="max">0.785398163397</param>
-                </command_interface>
-                <!-- <command_interface name="velocity">
-                    <param name="min">0.0</param>
-                    <param name="max">5.8178</param>
-                </command_interface> -->
-                <param name="initial_position">0.0</param>
-                <param name="max_velocity">5.8178</param>
+                    <param name="min">-0.7854</param>
+                    <param name="max">0.7854</param>
+                </command_interface>
+                <!-- <command_interface name="velocity">
+                    <param name="min">0.0</param>
+                    <param name="max">6.545</param>
+                </command_interface> -->
+                <param name="initial_position">0.0</param>
+                <param name="max_velocity">6.545</param>
                 <param name="max_effort">1.7</param>
             </joint>
@@ -84,13 +84,13 @@
                 <state_interface name="position" />
                 <command_interface name="position">
-                    <param name="min">-0.785398163</param>
-                    <param name="max">0.785398163397</param>
-                </command_interface>
-                <!-- <command_interface name="velocity">
-                    <param name="min">0.0</param>
-                    <param name="max">5.8178</param>
-                </command_interface> -->
-                <param name="initial_position">0.0</param>
-                <param name="max_velocity">5.8178</param>
+                    <param name="min">-0.7854</param>
+                    <param name="max">0.7854</param>
+                </command_interface>
+                <!-- <command_interface name="velocity">
+                    <param name="min">0.0</param>
+                    <param name="max">6.545</param>
+                </command_interface> -->
+                <param name="initial_position">0.0</param>
+                <param name="max_velocity">6.545</param>
                 <param name="max_effort">1.7</param>
             </joint>
@@ -98,13 +98,13 @@
                 <state_interface name="position" />
                 <command_interface name="position">
-                    <param name="min">-0.785398163</param>
-                    <param name="max">0.785398163397</param>
-                </command_interface>
-                <!-- <command_interface name="velocity">
-                    <param name="min">0.0</param>
-                    <param name="max">5.8178</param>
-                </command_interface> -->
-                <param name="initial_position">0.0</param>
-                <param name="max_velocity">5.8178</param>
+                    <param name="min">-0.7854</param>
+                    <param name="max">0.7854</param>
+                </command_interface>
+                <!-- <command_interface name="velocity">
+                    <param name="min">0.0</param>
+                    <param name="max">6.545</param>
+                </command_interface> -->
+                <param name="initial_position">0.0</param>
+                <param name="max_velocity">6.545</param>
                 <param name="max_effort">1.7</param>
             </joint>
@@ -113,14 +113,14 @@
                 <xacro:unless value="${enable_mimic}">
                     <command_interface name="position">
-                        <param name="min">-0.785398163</param>
-                        <param name="max">0.785398163397</param>
-                    </command_interface>
-                    <!-- <command_interface name="velocity">
-                        <param name="min">0.0</param>
-                        <param name="max">5.8178</param>
-                    </command_interface> -->
-                </xacro:unless>
-                <param name="initial_position">0.0</param>
-                <param name="max_velocity">5.8178</param>
+                        <param name="min">-0.7854</param>
+                        <param name="max">0.7854</param>
+                    </command_interface>
+                    <!-- <command_interface name="velocity">
+                        <param name="min">0.0</param>
+                        <param name="max">6.545</param>
+                    </command_interface> -->
+                </xacro:unless>
+                <param name="initial_position">0.0</param>
+                <param name="max_velocity">6.545</param>
                 <param name="max_effort">1.7</param>
                 <param name="mimic">ArFL_ThFL</param>
@@ -132,13 +132,13 @@
                 <state_interface name="position" />
                 <command_interface name="position">
-                    <param name="min">-0.785398163</param>
-                    <param name="max">0.785398163397</param>
-                </command_interface>
-                <!-- <command_interface name="velocity">
-                    <param name="min">0.0</param>
-                    <param name="max">5.8178</param>
-                </command_interface> -->
-                <param name="initial_position">0.0</param>
-                <param name="max_velocity">5.8178</param>
+                    <param name="min">-0.7854</param>
+                    <param name="max">0.7854</param>
+                </command_interface>
+                <!-- <command_interface name="velocity">
+                    <param name="min">0.0</param>
+                    <param name="max">6.545</param>
+                </command_interface> -->
+                <param name="initial_position">0.0</param>
+                <param name="max_velocity">6.545</param>
                 <param name="max_effort">1.7</param>
             </joint>
@@ -146,13 +146,13 @@
                 <state_interface name="position" />
                 <command_interface name="position">
-                    <param name="min">-0.785398163</param>
-                    <param name="max">0.785398163397</param>
-                </command_interface>
-                <!-- <command_interface name="velocity">
-                    <param name="min">0.0</param>
-                    <param name="max">5.8178</param>
-                </command_interface> -->
-                <param name="initial_position">0.0</param>
-                <param name="max_velocity">5.8178</param>
+                    <param name="min">-0.7854</param>
+                    <param name="max">0.7854</param>
+                </command_interface>
+                <!-- <command_interface name="velocity">
+                    <param name="min">0.0</param>
+                    <param name="max">6.545</param>
+                </command_interface> -->
+                <param name="initial_position">0.0</param>
+                <param name="max_velocity">6.545</param>
                 <param name="max_effort">1.7</param>
             </joint>
@@ -160,13 +160,13 @@
                 <state_interface name="position" />
                 <command_interface name="position">
-                    <param name="min">-0.785398163</param>
-                    <param name="max">0.785398163397</param>
-                </command_interface>
-                <!-- <command_interface name="velocity">
-                    <param name="min">0.0</param>
-                    <param name="max">5.8178</param>
-                </command_interface> -->
-                <param name="initial_position">0.0</param>
-                <param name="max_velocity">5.8178</param>
+                    <param name="min">-0.7854</param>
+                    <param name="max">0.7854</param>
+                </command_interface>
+                <!-- <command_interface name="velocity">
+                    <param name="min">0.0</param>
+                    <param name="max">6.545</param>
+                </command_interface> -->
+                <param name="initial_position">0.0</param>
+                <param name="max_velocity">6.545</param>
                 <param name="max_effort">1.7</param>
             </joint>
@@ -175,14 +175,14 @@
                 <xacro:unless value="${enable_mimic}">
                     <command_interface name="position">
-                        <param name="min">-0.785398163</param>
-                        <param name="max">0.785398163397</param>
-                    </command_interface>
-                    <!-- <command_interface name="velocity">
-                        <param name="min">0.0</param>
-                        <param name="max">5.8178</param>
-                    </command_interface> -->
-                </xacro:unless>
-                <param name="initial_position">0.0</param>
-                <param name="max_velocity">5.8178</param>
+                        <param name="min">-0.7854</param>
+                        <param name="max">0.7854</param>
+                    </command_interface>
+                    <!-- <command_interface name="velocity">
+                        <param name="min">0.0</param>
+                        <param name="max">6.545</param>
+                    </command_interface> -->
+                </xacro:unless>
+                <param name="initial_position">0.0</param>
+                <param name="max_velocity">6.545</param>
                 <param name="max_effort">1.7</param>
                 <param name="mimic">ArBR_ThBR</param>
@@ -194,13 +194,13 @@
                 <state_interface name="position" />
                 <command_interface name="position">
-                    <param name="min">-0.785398163</param>
-                    <param name="max">0.785398163397</param>
-                </command_interface>
-                <!-- <command_interface name="velocity">
-                    <param name="min">0.0</param>
-                    <param name="max">5.8178</param>
-                </command_interface> -->
-                <param name="initial_position">0.0</param>
-                <param name="max_velocity">5.8178</param>
+                    <param name="min">-0.7854</param>
+                    <param name="max">0.7854</param>
+                </command_interface>
+                <!-- <command_interface name="velocity">
+                    <param name="min">0.0</param>
+                    <param name="max">6.545</param>
+                </command_interface> -->
+                <param name="initial_position">0.0</param>
+                <param name="max_velocity">6.545</param>
                 <param name="max_effort">1.7</param>
             </joint>
@@ -208,13 +208,13 @@
                 <state_interface name="position" />
                 <command_interface name="position">
-                    <param name="min">-0.785398163</param>
-                    <param name="max">0.785398163397</param>
-                </command_interface>
-                <!-- <command_interface name="velocity">
-                    <param name="min">0.0</param>
-                    <param name="max">5.8178</param>
-                </command_interface> -->
-                <param name="initial_position">0.0</param>
-                <param name="max_velocity">5.8178</param>
+                    <param name="min">-0.7854</param>
+                    <param name="max">0.7854</param>
+                </command_interface>
+                <!-- <command_interface name="velocity">
+                    <param name="min">0.0</param>
+                    <param name="max">6.545</param>
+                </command_interface> -->
+                <param name="initial_position">0.0</param>
+                <param name="max_velocity">6.545</param>
                 <param name="max_effort">1.7</param>
             </joint>
@@ -222,13 +222,13 @@
                 <state_interface name="position" />
                 <command_interface name="position">
-                    <param name="min">-0.785398163</param>
-                    <param name="max">0.785398163397</param>
-                </command_interface>
-                <!-- <command_interface name="velocity">
-                    <param name="min">0.0</param>
-                    <param name="max">5.8178</param>
-                </command_interface> -->
-                <param name="initial_position">0.0</param>
-                <param name="max_velocity">5.8178</param>
+                    <param name="min">-0.7854</param>
+                    <param name="max">0.7854</param>
+                </command_interface>
+                <!-- <command_interface name="velocity">
+                    <param name="min">0.0</param>
+                    <param name="max">6.545</param>
+                </command_interface> -->
+                <param name="initial_position">0.0</param>
+                <param name="max_velocity">6.545</param>
                 <param name="max_effort">1.7</param>
             </joint>
@@ -237,14 +237,14 @@
                 <xacro:unless value="${enable_mimic}">
                     <command_interface name="position">
-                        <param name="min">-0.785398163</param>
-                        <param name="max">0.785398163397</param>
-                    </command_interface>
-                    <!-- <command_interface name="velocity">
-                        <param name="min">0.0</param>
-                        <param name="max">5.8178</param>
-                    </command_interface> -->
-                </xacro:unless>
-                <param name="initial_position">0.0</param>
-                <param name="max_velocity">5.8178</param>
+                        <param name="min">-0.7854</param>
+                        <param name="max">0.7854</param>
+                    </command_interface>
+                    <!-- <command_interface name="velocity">
+                        <param name="min">0.0</param>
+                        <param name="max">6.545</param>
+                    </command_interface> -->
+                </xacro:unless>
+                <param name="initial_position">0.0</param>
+                <param name="max_velocity">6.545</param>
                 <param name="max_effort">1.7</param>
                 <param name="mimic">ArBL_ThBL</param>
