Commit message: integration of hybrid control with cartesian space and joint space

File: src/DESCRIPTION/cerberus_v1/description/urdf/CERBERUS_V1.urdf (robot description, URDF)
Before this commit: robot CERBERUS_V1, 29 links, 28 joints
Links:
- link BODY: mass 1.0157 -> 0.88698
- link CAMERA: mass 0.29652 -> 0.30222
- link LIDAR: mass 0.10467 -> 0.10143
- link M: mass 0.25379 -> 0.26104
- link SeBL: mass 0.029079 -> 0.037021
- link SeBR: mass 0.029079 -> 0.037021
- link SeFL: mass 0.029079 -> 0.037021
- link SeFR: mass 0.029079 -> 0.037021
- link ShBL: mass 0.10028 -> 0.088995
- link ShBR: mass 0.10028 -> 0.088995
- link ShFL: mass 0.10028 -> 0.088995
- link ShFR: mass 0.10028 -> 0.088995
- link ThBL: mass 0.24964 -> 0.2297
- link ThBR: mass 0.24964 -> 0.2297
- link ThFL: mass 0.24964 -> 0.2297
- link ThFR: mass 0.24964 -> 0.2297
Joints:
- joint ArBL_ThBL: limit lower=-0.785398163397 upper=0.785398163397 effort=1.67 velocity=5.0 -> lower=-0.20944 upper=1.5708 effort=1.7 velocity=6.545; origin xyz=-0.050268 -0.027324 0.025077 rpy=-1.5708 0 -3.1416 -> xyz=-0.050268 -0.027324 0.025077 rpy=1.5708 -0.71 0
- joint ArBR_ThBR: limit lower=-0.785398163397 upper=0.785398163397 effort=1.67 velocity=5.0 -> lower=-1.5708 upper=0.20944 effort=1.7 velocity=6.545; origin xyz=0.050268 -0.027324 0.025223 rpy=-1.5708 0 3.1416 -> xyz=0.050268 -0.027324 0.025223 rpy=1.5708 0.71 0
- joint ArFL_ThFL: limit lower=-0.785398163397 upper=0.785398163397 effort=1.67 velocity=5.0 -> lower=-0.20944 upper=1.5708 effort=1.7 velocity=6.545; origin xyz=-0.050268 -0.027324 0.025077 rpy=-1.5708 0 -3.1416 -> xyz=-0.050268 -0.027324 0.025077 rpy=1.5708 -0.71 0
- joint ArFR_ThFR: limit lower=-0.785398163397 upper=0.785398163397 effort=1.67 velocity=5.0 -> lower=-1.5708 upper=0.20944 effort=1.7 velocity=6.545; origin xyz=0.050268 -0.027324 0.025223 rpy=-1.5708 0 3.1416 -> xyz=0.050268 -0.027324 0.025223 rpy=1.5708 0.71 0
- joint SeBL_M: axis 0.00011373 0 -1 -> 0 0 -1; limit lower=-0.785398163397 upper=0.785398163397 effort=1.67 velocity=5.0 -> lower=-0.7854 upper=0.7854 effort=1.7 velocity=6.545; origin xyz=-0.1154 0.095 0.044 rpy=0 -1.5707 -3.1416 -> xyz=-0.1154 0.095 0.044 rpy=1.5708 0 1.5708
- joint SeBR_M: axis 0.00011373 0 -1 -> 0 0 -1; limit lower=-0.785398163397 upper=0.785398163397 effort=1.67 velocity=5.0 -> lower=-0.7854 upper=0.7854 effort=1.7 velocity=6.545; origin xyz=-0.1154 -0.095 0.044 rpy=3.1416 1.5707 3.1416 -> xyz=-0.1154 -0.095 0.044 rpy=1.5708 0 1.5708
- joint SeFL_M: axis 0.00011373 0 -1 -> 0 0 -1; limit lower=-0.785398163397 upper=0.785398163397 effort=1.67 velocity=5.0 -> lower=-0.7854 upper=0.7854 effort=1.7 velocity=6.545; origin xyz=0.1446 0.095 0.044 rpy=0 -1.5707 -3.1416 -> xyz=0.1446 0.095 0.044 rpy=1.5708 0 1.5708
- joint SeFR_M: axis 0.00011373 0 -1 -> 0 0 -1; limit lower=-0.785398163397 upper=0.785398163397 effort=1.67 velocity=5.0 -> lower=-0.7854 upper=0.7854 effort=1.7 velocity=6.545; origin xyz=0.1446 -0.095 0.044 rpy=3.1416 1.5707 3.1416 -> xyz=0.1446 -0.095 0.044 rpy=1.5708 0 1.5708
- joint ShBL_ThBL: limit lower=-0.785398163397 upper=0.785398163397 effort=1.67 velocity=5.0 -> lower=-0.7854 upper=0.7854 effort=1.7 velocity=6.545; mimic joint=ArBL_ThBL multiplier=-0.304 offset=0 -> joint=ArBL_ThBL multiplier=-0.2824 offset=0; origin xyz=-0.18101 0.0059195 0.01015 rpy=0 0 1.3090 -> xyz=-0.18101 0.0059195 0.01015 rpy=0 0 1.0
- joint ShBR_ThBR: limit lower=-0.785398163397 upper=0.785398163397 effort=1.67 velocity=5.0 -> lower=-0.7854 upper=0.7854 effort=1.7 velocity=6.545; mimic joint=ArBR_ThBR multiplier=-0.304 offset=0 -> joint=ArBR_ThBR multiplier=-0.2824 offset=0; origin xyz=0.18101 0.0059195 0.01015 rpy=0 0 -1.3090 -> xyz=0.18101 0.0059195 0.01015 rpy=0 0 -1.0
- joint ShFL_ThFL: limit lower=-0.785398163397 upper=0.785398163397 effort=1.67 velocity=5.0 -> lower=-0.7854 upper=0.7854 effort=1.7 velocity=6.545; mimic joint=ArFL_ThFL multiplier=-0.304 offset=0 -> joint=ArFL_ThFL multiplier=-0.2824 offset=0; origin xyz=-0.18101 0.0059195 0.01015 rpy=0 0 1.3090 -> xyz=-0.18101 0.0059195 0.01015 rpy=0 0 1.0
- joint ShFR_ThFR: limit lower=-0.785398163397 upper=0.785398163397 effort=1.67 velocity=5.0 -> lower=-0.7854 upper=0.7854 effort=1.7 velocity=6.545; mimic joint=ArFR_ThFR multiplier=-0.304 offset=0 -> joint=ArFR_ThFR multiplier=-0.2824 offset=0; origin xyz=0.18101 0.0059195 0.01015 rpy=0 0 -1.3090 -> xyz=0.18101 0.0059195 0.01015 rpy=0 0 -1.0
- joint ThBL_SeBL: limit lower=-0.785398163397 upper=0.785398163397 effort=1.67 velocity=5.0 -> lower=-0.7854 upper=0.7854 effort=1.7 velocity=6.545; origin xyz=2.2896E-05 -0.0144 0.045901 rpy=1.5708 -0.70743 0 -> xyz=0.0144 2.8116E-05 0.045901 rpy=1.5708 -1.2 1.5708
- joint ThBR_SeBR: limit lower=-0.785398163397 upper=0.785398163397 effort=1.67 velocity=5.0 -> lower=-0.7854 upper=0.7854 effort=1.7 velocity=6.545; origin xyz=2.2896E-05 -0.0144 0.045901 rpy=1.5708 0.70743 0 -> xyz=-0.0144 -2.8116E-05 0.045901 rpy=1.5708 1.2 -1.5708
- joint ThFL_SeFL: limit lower=-0.785398163397 upper=0.785398163397 effort=1.67 velocity=5.0 -> lower=-0.7854 upper=0.7854 effort=1.7 velocity=6.545; origin xyz=2.2896E-05 -0.0144 0.045901 rpy=1.5708 -0.70743 0 -> xyz=0.0144 2.8116E-05 0.045901 rpy=1.5708 -1.35 1.5708
- joint ThFR_SeFR: limit lower=-0.785398163397 upper=0.785398163397 effort=1.67 velocity=5.0 -> lower=-0.7854 upper=0.7854 effort=1.7 velocity=6.545; origin xyz=2.2896E-05 -0.0144 0.045901 rpy=1.5708 0.70743 0 -> xyz=-0.0144 -2.8116E-05 0.045901 rpy=1.5708 1.35 -1.5708
